File: CircuitoGeneral/espirometro.kicad_sch (KiCad schematic)
At the start: 42 parts, among them J1 Sensor Diferencial de Presión, J10 Convertidor de voltaje, J11 Entrada de +5V, J12 TEMP, J13 PIM, J14 DP, J15 Pantalla LCD, J16 DF_PLAYER, J17 MICROSD, J18 TEMP, J19 Salida DP, J2 Salida PIM, J20 Alimentación, J3 Salida TEMP, J4 ALIMENTACIÓN, J5 Audio, J6 Audio, J7 3.3V, J8 5V, J9 Convertidor de Voltaje, U1 LM358, U2 LM358, U4 ESP32

Commit message: Actualización de esquemático y PCB de KiCad
Parts:
- removed J15: Pantalla LCD, Connector_PinSocket_2.54mm:PinSocket_1x14_P2.54mm_Vertical, symbol Connector:Conn_01x14_Pin
- added J21: Pantalla LCD, Connector_PinSocket_2.54mm:PinSocket_1x14_P2.54mm_Vertical, symbol Connector:Conn_01x14_Pin
Connections:
- net +5V: now also J21.1 (Pin_1)
- net 3,3V: now also J21.8 (Pin_8)
- net CS: now also J21.3 (Pin_3)
- net D/C: now also J21.5 (Pin_5)
- net GND: now also J21.2 (Pin_2)
- net GPIO21: now also J21.6 (Pin_6)
- net GPIO22: now also J21.7 (Pin_7)
- net GPIO25: now also J21.12 (Pin_12)
- net GPIO26: now also J21.13 (Pin_13)
- net GPIO32: now also J21.10 (Pin_10)
- net GPIO33: now also J21.11 (Pin_11)
- net GPIO4: now also J21.4 (Pin_4)
- net MISO: now also J21.9 (Pin_9)
