File: ESP_SD_PANTALLA/ESP_SD_PANTALLA.kicad_sch (KiCad schematic)
At the start: 10 parts, among them J1 ALIMENTACIÓN, J2 3.3V, J3 5V, J4 TEMP, J5 PIM, J6 DP, J7 DF_PLAYER, J8 MICROSD, J9 Pantalla LCD, U1 ESP32

Commit message: Actualización de esquemático y PCB de KiCad
Connections:
- net GPIO17: no longer J9.6 (Pin_6)
- net GPIO18: no longer J9.7 (Pin_7)
- net GPIO21: now also J9.6 (Pin_6)
- net GPIO22: now also J9.7 (Pin_7)
Changed lines of the file:
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@@
 		)
 	)
-	(label "GPIO18"
+	(label "GPIO22"
 		(at 176.53 187.96 0)
 		(effects
@@
 		)
 	)
-	(label "GPIO17"
+	(label "GPIO21"
 		(at 176.53 185.42 0)
 		(effects
