File: ESP_SD_PANTALLA/ESP_SD_PANTALLA.kicad_pcb (KiCad board)
At the start: 2 copper layers, 74 x 77 mm, 10 parts, among them J1 ALIMENTACIÓN, J2 3.3V, J3 5V, J4 TEMP, J5 PIM, J6 DP, J7 DF_PLAYER, J8 MICROSD, J9 Pantalla LCD, U1 ESP32

Commit message: Actualización de esquemático y PCB de KiCad
Connections:
- J9 pad 6: /GPIO17 -> /GPIO21
- J9 pad 7: /GPIO18 -> /GPIO22
Routing:
- net /GPIO21: track 11.7 -> 118.8 mm
- net /GPIO22: track 8.50 -> 113.9 mm
- net /GPIO17: track 96.9 -> 0.00 mm
- net /GND: track 239.1 -> 334.9 mm, vias 2 -> 4
- net /GPIO18: track 91.4 -> 0.00 mm
- net /GPIO13: track 7.53 -> 12.7 mm
Other:
- board outline removed
