File: PIM_ESPIROMETRIA/PIM_ESPIROMETRIA.kicad_pcb (KiCad board)
At the start: 2 copper layers, 70 x 80.5 mm, 23 parts, among them J1 DP, J2 Salida PIM, J3 Salida TEMP, J4 TEMP, J5 Salida DP, J9 Alimentación, U1 LM358

Commit message: Actualiza todos los archivos
Parts:
- added C11: 100nF, Capacitor_THT:C_Disc_D5.0mm_W2.5mm_P2.50mm, F.Cu at (1.52, 1.52)
- added C12: 100nF, Capacitor_THT:C_Disc_D5.0mm_W2.5mm_P2.50mm, F.Cu at (1.52, 5.58)
- added C13: 100nF, Capacitor_THT:C_Disc_D5.0mm_W2.5mm_P2.50mm, F.Cu at (1.52, 9.62)
- added R19: 1k, Resistor_THT:R_Axial_DIN0204_L3.6mm_D1.6mm_P7.62mm_Horizontal, F.Cu at (7.53, 1.07)
- added R20: 1k, Resistor_THT:R_Axial_DIN0204_L3.6mm_D1.6mm_P7.62mm_Horizontal, F.Cu at (7.53, 4.22)
- added U1: MCP6004, Package_DFN_QFN:DFN-8-1EP_3x2mm_P0.5mm_EP1.75x1.45mm, F.Cu at (8.90, 7.73)
- J1: value DP -> Sensor Diferencial de Presión
- R3: value 2.4k -> 12.4k
- R6: value R -> 511
- renumbered U5 to SensorPIM1
Connections:
- J5 pad 1: /DP -> /GPIO36
- R2 pad 2: Net-(U1A-+) -> Net-(U1C-+)
- R4 pad 1: Net-(U1B-+) -> Net-(U1A-+)
- R5 pad 2: Net-(U1B-+) -> Net-(U1A-+)
- U4 pad 4: /GPIO39 -> /PIM/PEM
- U4 pad 5: /1.65V -> /2.5V
- U4 pad 6: /-5V -> /GND
- U6 pad 6: /-5V -> /GND
