File: PIM_ESPIROMETRIA/PIM_ESPIROMETRIA.kicad_sch (KiCad schematic)
At the start: 23 parts, among them J1 Sensor Diferencial de Presión, J2 Salida PIM, J3 Salida TEMP, J4 TEMP, J5 Salida DP, J9 Alimentación, U1 LM358

Commit message: Actualiza todos los archivos
Parts:
- removed C3, C4, C5, C6, C7: 100nF, Capacitor_THT:C_Disc_D5.0mm_W2.5mm_P2.50mm, symbol Device:C
- removed U1: LM358, Package_DIP:DIP-8_W7.62mm, symbol Amplifier_Operational:LM358
- added C10, C8: 100n, symbol Device:C
- added C12, C13, C15: 100nF, Capacitor_THT:C_Disc_D5.0mm_W2.5mm_P2.50mm, symbol Device:C
- added R10: 39k, symbol Device:R
- added R11, R13, R21, R7: 75k, symbol Device:R
- added R15: 1K, symbol Device:R
- added R16: 3.2K, symbol Device:R
- added R19: 4.7k, Resistor_THT:R_Axial_DIN0204_L3.6mm_D1.6mm_P7.62mm_Horizontal, symbol Device:R
- added R20: 1k, Resistor_THT:R_Axial_DIN0204_L3.6mm_D1.6mm_P7.62mm_Horizontal, symbol Device:R
- added R22, R9: 5k, symbol Device:R
- added U1, U2, U3: TL082, symbol Amplifier_Operational:TL082
- R3: value 2.4k -> 5k
- R6: value R -> 5k
- renumbered U5 to SensorPIM1
Connections:
- net -5V: no longer U4.6 (VS-), U6.6 (VS-)
- net 1.65V: now also R15.1, U1.1, U1.2 (-); no longer U6.5 (Vref)
- net 3.3V: now also C12.2, C13.1, C15.2, U1.8 (V+), U2.8 (V+), U3.8 (V+)
- net DP: now also R11.1, U2.1, U2.2 (-); no longer J5.1 (Pin_1)
- net GND: now also U4.6 (VS-), U6.6 (VS-), C10.2, C12.1, C13.2, C8.2, R20.2, U1.4 (V-), U2.4 (V-), U2.5 (+)
- net GPIO39: now also R16.2, U3.7; no longer U4.4 (OUT)
- net at R4.1, R5.2: now also U1.3 (+)
- net at C2.2, R1.2, R2.1: no longer C1.1
- net at R2.2: now also C1.1, U2.3 (+)
- net GPIO07 renamed GPIO02
- new net: R22.2, R9.1
- new net: R10.2, R9.2, U3.2 (-)
- new net: R15.2, R16.1, U3.6 (-)
- new net: R19.2, R20.1, U1.5 (+)
- new net: R13.1, R21.2
- new net: R11.2, R7.1
- new net: C8.1, R7.2, U3.3 (+)
- new net: U2.6 (-), U2.7
- new net 1V: R22.1, U1.6 (-), U1.7, U6.5 (Vref)
- new net 5V: R19.1
- new net GPIO36: J5.1 (Pin_1), R10.1, U3.1
- new net PIM/PEM: R21.1, U4.4 (OUT)
- new net VIN: C10.1, R13.2, U3.5 (+)
Other:
- moved on the sheet: C2, J1, J2, J3, J4, J5, J9, R1, R2, R3, R4, R5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
